File: pcb/KickerKast/KickerKast.sch (KiCad schematic (older format))
At the start: 29 parts, among them CON1 BARREL_JACK, P1 SENS1, P2 SENS2, P3 Program, P4 UART, P5 7SEG_1, P6 7SEG_2, Q1 7S1a, Q2 7S1b, Q3 7S2a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

Commit message: added extra connector to kickerkast pcb
Parts:
- added P7: CONN_01X05, Pin_Headers:Pin_Header_Straight_1x05, symbol CONN_01X05
Connections:
- net RC0: now reaches U1.11 (RC0/T1OSO/T13CKI)
- net RC0: now also P7.5 (P5)
- net RC1: now reaches U1.12 (RC1/T1OSI/CCP2/UOE)
- net RC1: now also P7.4 (P4)
- net RC2: now reaches U1.13 (RC2/CCP1)
- net RC2: now also P7.3 (P3)
- net RC4: now reaches U1.15 (RC4/D-/VM)
- net RC4: now also P7.2 (P2)
- net RC5: now reaches U1.16 (rc5/D+/VP)
- net RC5: now also P7.1 (P1)

Commit message: description
Parts:
- C1, C2, C4: symbol C -> Device:C
- C3: symbol CP -> Device:CP
- CON1: symbol BARREL_JACK -> KickerKast-rescue:BARREL_JACK
- D1: symbol LED -> KickerKast-rescue:LED
- P1, P2, P5, P6: symbol CONN_02X05 -> KickerKast-rescue:CONN_02X05
- P3: symbol CONN_01X06 -> KickerKast-rescue:CONN_01X06
- P4: symbol CONN_01X04 -> KickerKast-rescue:CONN_01X04
- P7: symbol CONN_01X05 -> KickerKast-rescue:CONN_01X05
- Q1, Q2, Q3, Q4: symbol BC547 -> KickerKast-rescue:BC547
- R1, R10, R2, R3, R4, R5, R6, R7, R8, R9: symbol R -> Device:R
- SW1: symbol SW_PUSH -> KickerKast-rescue:SW_PUSH
- U1: symbol PIC18F2550 -> KickerKast-rescue:PIC18F2550
- Y1: symbol Crystal -> Device:Crystal
